Commit message: renaming bard_urdf to barrett_urdf

File: barrett_urdf/models/arm.urdf.xacro (robot description, xacro)
@@ -24,7 +24,7 @@
 -->
 <robot xmlns:xacro="http://www.ros.org/wiki/xacro">
-  <include filename="$(find bard_urdf)/models/hand.urdf.xacro"/>
-  <include filename="$(find bard_urdf)/models/common.urdf.xacro"/>
-  <include filename="$(find bard_urdf)/models/components.urdf.xacro"/>
+  <include filename="$(find barrett_urdf)/models/hand.urdf.xacro"/>
+  <include filename="$(find barrett_urdf)/models/common.urdf.xacro"/>
+  <include filename="$(find barrett_urdf)/models/components.urdf.xacro"/>
   <!-- different types of arms -->
   <xacro:macro name="wam_4dof" params="prefix parentLink xyz rpy">

File: barrett_urdf/models/common.urdf.xacro (robot description, xacro)
@@ -31,5 +31,5 @@
   xmlns:xacro="http://ros.org/wiki/xacro">
   <!-- Directories -->
-  <xacro:property name="homeDirectory" value="package://bard_urdf" />
+  <xacro:property name="homeDirectory" value="package://barrett_urdf" />
   <xacro:property name="highResModelDirectory" value="${homeDirectory}/models/componentSTL/splitModels" />
   <!-- Constants -->

File: barrett_urdf/models/components.urdf.xacro (robot description, xacro)
@@ -30,6 +30,6 @@
   xmlns:geom="http://playerstage.sourceforge.net/gazebo/xmlschema/#geom"
   xmlns:xacro="http://ros.org/wiki/xacro">
-  <include filename="$(find bard_urdf)/models/hand.urdf.xacro"/>
-  <include filename="$(find bard_urdf)/models/common.urdf.xacro"/>
+  <include filename="$(find barrett_urdf)/models/hand.urdf.xacro"/>
+  <include filename="$(find barrett_urdf)/models/common.urdf.xacro"/>
   <!-- Upper arm macros -->
   <xacro:macro name="Shoulder" params="prefix parentLink xyz rpy">

File: barrett_urdf/models/hand.urdf.xacro (robot description, xacro)
@@ -28,5 +28,5 @@
   xmlns:interface="http://playerstage.sourceforge.net/gazebo/xmlschema/#interface"
   xmlns:xacro="http://www.ros.org/wiki/xacro">
-  <include filename="$(find bard_urdf)/models/common.urdf.xacro"/>
+  <include filename="$(find barrett_urdf)/models/common.urdf.xacro"/>
   <!-- Palm -->
   <xacro:macro name="Palm" params="prefix">

File: barrett_urdf/models/left_arm.urdf.xacro (robot description, xacro)
@@ -29,9 +29,9 @@
   xmlns:controller="http://playerstage.sourceforge.net/gazebo/xmlschema/#controller">
   <!-- Some macros used by the WAM urdf -->
-  <include filename="$(find bard_urdf)/models/common.urdf.xacro"/>
+  <include filename="$(find barrett_urdf)/models/common.urdf.xacro"/>
   <!-- Definition of a single WAM arm -->
-  <include filename="$(find bard_urdf)/models/arm.urdf.xacro"/>
+  <include filename="$(find barrett_urdf)/models/arm.urdf.xacro"/>
   <!-- Definition of all the different parts of a WAM arm -->
-  <include filename="$(find bard_urdf)/models/components.urdf.xacro"/>
+  <include filename="$(find barrett_urdf)/models/components.urdf.xacro"/>
   <!-- Materials -->
   <material name="WAMGrey">

File: barrett_urdf/models/two_arms_example.urdf.xacro (robot description, xacro)
@@ -26,7 +26,7 @@
   xmlns:xacro="http://www.ros.org/wiki/xacro"
   xmlns:controller="http://playerstage.sourceforge.net/gazebo/xmlschema/#controller">
-  <include filename="$(find bard_urdf)/models/common.urdf.xacro"/>
-  <include filename="$(find bard_urdf)/models/arm.urdf.xacro"/>
-  <include filename="$(find bard_urdf)/models/components.urdf.xacro"/>
+  <include filename="$(find barrett_urdf)/models/common.urdf.xacro"/>
+  <include filename="$(find barrett_urdf)/models/arm.urdf.xacro"/>
+  <include filename="$(find barrett_urdf)/models/components.urdf.xacro"/>
   <!-- Materials -->
   <material name="WAMGrey">
@@ -46,5 +46,5 @@
         <geometry>
           <!--box size="0.04 2.54 0.04"/-->
-          <mesh filename="package://bard_urdf/models/componentSTL/bench_lattice.dae"/>
+          <mesh filename="package://barrett_urdf/models/componentSTL/bench_lattice.dae"/>
         </geometry>
       </visual>
@@ -52,5 +52,5 @@
         <origin xyz="0 0 0" rpy="0 0 0" />
         <geometry>
-          <mesh filename="package://bard_urdf/models/componentSTL/bench_lattice.stl"/>
+          <mesh filename="package://barrett_urdf/models/componentSTL/bench_lattice.stl"/>
         </geometry>
       </collision>
