Commit message: calibration script

File: barrett_model/models/components.urdf.xacro (robot description, xacro)
@@ -39,5 +39,5 @@
       <origin xyz="${xyz}" rpy="${rpy}"/>
       <axis xyz="0 -1 0"/>
-      <limit effort="30" lower="-2.6" upper="2.6" velocity="0.50"/>
+      <limit effort="40" lower="-2.6" upper="2.6" velocity="0.50"/>
       <!-- <safety_controller k_position="10000000" k_velocity="10000000" soft_lower_limit="-100.0" soft_upper_limit="100.0" /> -->
       <dynamics damping="1.0" friction="100.0"/>
@@ -77,5 +77,5 @@
       <origin xyz="0 0 0" rpy="${0.5 * PI} 0 0"/>
       <axis xyz="0 1 0"/>
-      <limit effort="30" lower="-1.985" upper="1.985" velocity="0.5"/>
+      <limit effort="40" lower="-1.985" upper="1.985" velocity="0.5"/>
       <!-- <safety_controller k_position="100" k_velocity="3" soft_lower_limit="-100.0" soft_upper_limit="100.0" /> -->
       <dynamics damping="1.0" friction="100.0"/>
@@ -228,5 +228,5 @@
       <origin xyz="0.045 -0.55 0" rpy="${0.5 * PI} 0 0"/>
       <axis xyz="0 1 0"/>
-      <limit effort="15" lower="-0.9" upper="${PI}" velocity="0.20"/>
+      <limit effort="25" lower="-0.9" upper="${PI}" velocity="0.20"/>
       <!-- <safety_controller k_position="100" k_velocity="3" soft_lower_limit="-100.0" soft_upper_limit="100.0" /> -->
       <dynamics damping="1.0" friction="100.0"/>

Commit message: calibration working, post-tensioning

File: barrett_model/models/components.urdf.xacro (robot description, xacro)
@@ -39,5 +39,5 @@
       <origin xyz="${xyz}" rpy="${rpy}"/>
       <axis xyz="0 -1 0"/>
-      <limit effort="40" lower="-2.6" upper="2.6" velocity="0.50"/>
+      <limit effort="60" lower="-2.6" upper="2.6" velocity="0.50"/>
       <!-- <safety_controller k_position="10000000" k_velocity="10000000" soft_lower_limit="-100.0" soft_upper_limit="100.0" /> -->
       <dynamics damping="1.0" friction="100.0"/>
@@ -190,5 +190,5 @@
       <origin xyz="-0.045 0 .35" rpy="-${0.5 * PI} 0 ${0.5 * PI}"/>
       <axis xyz="0 -1 0"/>
-      <limit effort="5" lower="-4.8" upper="1.3" velocity="0.20"/>
+      <limit effort="5" lower="-4.8" upper="1.3" velocity="0.80"/>
       <!-- <safety_controller k_position="100" k_velocity="3" soft_lower_limit="-100.0" soft_upper_limit="100.0" /> -->
       <dynamics damping="1.0" friction="100.0"/>
@@ -228,5 +228,5 @@
       <origin xyz="0.045 -0.55 0" rpy="${0.5 * PI} 0 0"/>
       <axis xyz="0 1 0"/>
-      <limit effort="25" lower="-0.9" upper="${PI}" velocity="0.20"/>
+      <limit effort="25" lower="-0.9" upper="${PI}" velocity="0.80"/>
       <!-- <safety_controller k_position="100" k_velocity="3" soft_lower_limit="-100.0" soft_upper_limit="100.0" /> -->
       <dynamics damping="1.0" friction="100.0"/>
@@ -266,5 +266,5 @@
       <origin xyz="-0.045 0 .3" rpy="-${0.5 * PI} 0 ${0.5 * PI}"/>
       <axis xyz="0 -1 0"/>
-      <limit effort="5" lower="-4.8" upper="1.3" velocity="0.20"/>
+      <limit effort="5" lower="-4.8" upper="1.3" velocity="0.80"/>
       <!-- <safety_controller k_position="100" k_velocity="3" soft_lower_limit="-100.0" soft_upper_limit="100.0" /> -->
       <dynamics damping="1.0" friction="100.0"/>
@@ -303,5 +303,5 @@
       <origin xyz="0 0 0" rpy="${0.5 * PI} ${PI} 0"/>
       <axis xyz="0 1 0"/>
-      <limit effort="5" lower="-1.45" upper="1.45" velocity="0.20"/><!-- 1.45 is a limit taken in from 1.5 due to saftey and differences between arms. -->
+      <limit effort="5" lower="-1.45" upper="1.45" velocity="0.80"/><!-- 1.45 is a limit taken in from 1.5 due to saftey and differences between arms. -->
       <!-- <safety_controller k_position="100" k_velocity="3" soft_lower_limit="-100.0" soft_upper_limit="100.0" /> -->
       <dynamics damping="1.0" friction="100.0"/>
